File: design/dc-load/dc-load.kicad_sch (KiCad schematic)
At the start: 65 parts, among them Q1 Q_NMOS_GDS, U1 LT1636IN8PBF, U2 LT1636IN8PBF, U3 LT1636IN8PBF, U4 STM32F030RCTx

Commit message: add docs
Parts:
- removed SW? (x2): SW_Push, symbol Switch:SW_Push
Connections:
- net GND: now also U4.12 (VSSA), U4.18 (VSS), U4.31 (VSS), U4.47 (VSS), U4.60 (BOOT0), U4.63 (VSS)
- net RESET: now also U4.7 (NRST)
Other:
- moved on the sheet: D2, R25
